File: IsoISE-feather.kicad_pcb (KiCad board)
At the start: 2 copper layers, 50.8 x 22.9 mm, 119 parts, among them J1 Conn_01x03, J2 BNC, J3 FEATHER, U1 MTU1D0305MC, U2 ADUM1250ARZ, U3 MCP4017, U4 TL072, U5 REF3130, U6 MCP3221

Commit message: tweaked silkscreen and replaced bnc to get 3d model..
Parts:
- J2: footprint kicad-library:BNC-Amphenol -> kicad-library:BNC_Socket_Gmod
- moved J2 7.05 mm to (134.2, 105.5), turned to 90 degrees
- moved G*** 4.50 mm to (163.5, 102.7)
- moved REF** 0.58 mm to (136.9, 111.2)
- moved REF** 0.58 mm to (138.5, 106.6)
- moved REF** 0.29 mm to (133.0, 99.7)
- moved REF** 0.22 mm to (133.1, 109.9)
- moved REF** 0.17 mm to (136.5, 101.6)
Other:
- outline, holes or cut-outs redrawn

Commit message: files as submitted to oshpark
Parts:
- moved J1 0.42 mm to (170.6, 110.4)
- moved REF** 0.27 mm to (172.5, 109.6)
- moved REF** 0.25 mm to (172.4, 107.0)
- moved REF** 0.19 mm to (172.4, 104.2)
Routing:
- net Net-(C5-Pad2): track 29.1 -> 30.5 mm

Commit message: updated logo on board
Parts:
- REF***: footprint Symbols:KiCad-Logo2_6mm_SilkScreen -> Symbols:Symbol_KiCAD-Logo_CopperAndSilkScreenTop
